File: Starter/KC47852.kicad_pcb (KiCad board)
At the start: 2 copper layers, 114.3 x 88.9 mm, 50 parts, among them J1 AudioJack, J2 Speaker, J3 UART1, J4 Pot, J6 GND, J7 DACOUT, SW1 UP, SW2 LEFT, SW3 DOWN, SW4 RGHT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

Commit message: Minor changes!
Parts:
- removed TP1: 3.3V, ECE319K:Testpoint_1x02_P2.54mm
- removed U1: Adafruit ST7735R, ECE319K:adafruit_st7735r
- added J8: Conn_01x05_Pin, Connector_PinHeader_2.54mm:PinHeader_1x05_P2.54mm_Vertical, F.Cu at (29.6, 49.3)
- J1: value AudioJack -> Conn_01x09_Pin; footprint ECE319K:Jack_3.5mm_CUI_SJ1-3523N_Horizontal -> Connector_PinHeader_2.54mm:PinHeader_1x09_P2.54mm_Vertical
- U5: footprint ECE319K:DIP-16_W7.62mm -> ECE319H:DIP-16_W7.62mm
- moved J3 52.7 mm to (106.3, 69.6)
- moved U4 37.0 mm to (223.2, 78.3)
- moved J1 4.89 mm to (24.9, 49.3), turned to 0 degrees
Connections:
- C1 pad 1: unconnected-(C1-Pad1) -> Net-(U3-FC1)
- C1 pad 2: unconnected-(C1-Pad2) -> GND
- C2 pad 1: unconnected-(C2-Pad1) -> Net-(U3-FC2)
- C2 pad 2: unconnected-(C2-Pad2) -> GND
- C3 pad 1: unconnected-(C3-Pad1) -> DACOUT
- C3 pad 2: unconnected-(C3-Pad2) -> Net-(C3-Pad2)
- C4 pad 1: unconnected-(C4-Pad1) -> +3V3
- C4 pad 2: unconnected-(C4-Pad2) -> Net-(U6-Gnd)
- D1 pad 1: unconnected-(D1-K-Pad1) -> GND
- D1 pad 2: unconnected-(D1-A-Pad2) -> Net-(D1-A)
- D2 pad 1: unconnected-(D2-K-Pad1) -> GND
- D2 pad 2: unconnected-(D2-A-Pad2) -> Net-(D2-A)
- D3 pad 1: unconnected-(D3-K-Pad1) -> GND
- D3 pad 2: unconnected-(D3-A-Pad2) -> Net-(D3-A)
- D4 pad 1: unconnected-(D4-K-Pad1) -> Net-(D4-K)
- D4 pad 2: unconnected-(D4-A-Pad2) -> Net-(D4-A)
- J2 pad 1: unconnected-(J2-Pad1) -> Net-(U3-VO1)
- J2 pad 2: unconnected-(J2-Pad2) -> Net-(U3-VO2)
- J4 pad 1: unconnected-(J4-A-Pad1) -> PB18
- J4 pad 2: unconnected-(J4-B-Pad2) -> PB18
- J7 pad 1: unconnected-(J7-A-Pad1) -> DACOUT
- J7 pad 2: unconnected-(J7-B-Pad2) -> DACOUT
- JP1 pad 1: unconnected-(JP1-A-Pad1) -> DACOUT
- JP1 pad 3: unconnected-(JP1-B-Pad3) -> PB18
- R1 pad 1: unconnected-(R1-Pad1) -> PA28
- R1 pad 2: unconnected-(R1-Pad2) -> Net-(D1-A)
- R10 pad 1: unconnected-(R10-Pad1) -> DACOUT
- R10 pad 2: unconnected-(R10-Pad2) -> PB1
- R11 pad 1: unconnected-(R11-Pad1) -> DACOUT
- R11 pad 2: unconnected-(R11-Pad2) -> PB0
- R12 pad 1: unconnected-(R12-Pad1) -> PB24
- R12 pad 2: unconnected-(R12-Pad2) -> GND
- R13 pad 1: unconnected-(R13-Pad1) -> PB23
- R13 pad 2: unconnected-(R13-Pad2) -> GND
- R14 pad 1: unconnected-(R14-Pad1) -> PA16
- R14 pad 2: unconnected-(R14-Pad2) -> GND
- R15 pad 1: unconnected-(R15-Pad1) -> PA15
- R15 pad 2: unconnected-(R15-Pad2) -> GND
- R16 pad 1: unconnected-(R16-Pad1) -> Net-(U3-VO1)
- R16 pad 2: unconnected-(R16-Pad2) -> Net-(U3-VIN)
- R17 pad 1: unconnected-(R17-Pad1) -> Net-(U3-VIN)
- R17 pad 2: unconnected-(R17-Pad2) -> Net-(C3-Pad2)
- R18 pad 1: unconnected-(R18-Pad1) -> +5V
- R18 pad 2: unconnected-(R18-Pad2) -> Net-(D4-A)
- R2 pad 1: unconnected-(R2-Pad1) -> PA27
- R2 pad 2: unconnected-(R2-Pad2) -> Net-(D2-A)
- R3 pad 1: unconnected-(R3-Pad1) -> PA26
- R3 pad 2: unconnected-(R3-Pad2) -> Net-(D3-A)
- R4 pad 1: unconnected-(R4-Pad1) -> DACOUT
- R4 pad 2: unconnected-(R4-Pad2) -> PB4
- R5 pad 1: unconnected-(R5-Pad1) -> DACOUT
- R5 pad 2: unconnected-(R5-Pad2) -> PB4
- R6 pad 1: unconnected-(R6-Pad1) -> DACOUT
- R6 pad 2: unconnected-(R6-Pad2) -> PB3
- R7 pad 1: unconnected-(R7-Pad1) -> Net-(R7-Pad1)
- R7 pad 2: unconnected-(R7-Pad2) -> PB2
- R8 pad 1: unconnected-(R8-Pad1) -> DACOUT
- R8 pad 2: unconnected-(R8-Pad2) -> Net-(R7-Pad1)
- R9 pad 1: unconnected-(R9-Pad1) -> DACOUT
- R9 pad 2: unconnected-(R9-Pad2) -> PB1
- RV1 pad 1: unconnected-(RV1-Pad1) -> GND
- RV1 pad 2: unconnected-(RV1-Pad2) -> PB18
- RV1 pad 3: unconnected-(RV1-Pad3) -> +3V3
- SW1 pad 1: unconnected-(SW1-Pad1) -> PB24
- SW1 pad 2: unconnected-(SW1-Pad2) -> +3V3
- SW2 pad 1: unconnected-(SW2-Pad1) -> PB23
- SW2 pad 2: unconnected-(SW2-Pad2) -> +3V3
- SW3 pad 1: unconnected-(SW3-Pad1) -> PA16
- SW3 pad 2: unconnected-(SW3-Pad2) -> +3V3
- SW4 pad 1: unconnected-(SW4-Pad1) -> PA15
- SW4 pad 2: unconnected-(SW4-Pad2) -> +3V3
- U3 pad 2: unconnected-(U3-FC2-Pad2) -> Net-(U3-FC2)
- U3 pad 3: unconnected-(U3-FC1-Pad3) -> Net-(U3-FC1)
- U3 pad 4: unconnected-(U3-VIN-Pad4) -> Net-(U3-VIN)
- U3 pad 5: unconnected-(U3-VO1-Pad5) -> Net-(U3-VO1)
- U3 pad 6: unconnected-(U3-Vcc-Pad6) -> +5V
- U3 pad 7: unconnected-(U3-GND-Pad7) -> GND
- U3 pad 8: unconnected-(U3-VO2-Pad8) -> Net-(U3-VO2)
- U4 pad 15: +3V3 -> Net-(U4-LED+)
- U4 pad 2: +3V3 -> Net-(U4-LED+)
- U4 pad 6: PB15 -> PB13
- U5 pad 1: unconnected-(U5-1B-Pad1) -> PA8
- U5 pad 16: unconnected-(U5-1C-Pad16) -> Net-(D4-K)
- U5 pad 8: unconnected-(U5-E-Pad8) -> GND
- U6 pad 1: unconnected-(U6-Gnd-Pad1) -> Net-(U6-Gnd)
- U6 pad 2: unconnected-(U6-Vs-Pad2) -> +3V3
- U6 pad 3: unconnected-(U6-Out-Pad3) -> PA22

Commit message: Minor edits V2!
Parts:
- moved U4 128.0 mm to (136.4, -15.8)
- moved RV1 57.0 mm to (118.9, 118.5)
Changed lines of the file:
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@@
 	(footprint "ECE319K:PTA2043pot"
 		(layer "F.Cu")
-		(at 171.565 140.49)
+		(at 118.905 118.55)
 		(descr "Bourns single-gang slide potentiometer, 20.0mm travel, https://www.bourns.com/docs/Product-Datasheets/pta.pdf")
 		(tags "Bourns single-gang slide potentiometer 20.0mm")
@@
 	(footprint "ECE319K:hiletgo_st7735r"
 		(layer "F.Cu")
-		(at 223.225001 78.270526)
+		(at 136.400001 -15.804474)
 		(property "Reference" "U4"
 			(at -12.7 24.765 0)
