File: Starter/KC47852.kicad_pcb (KiCad board)
At the start: 2 copper layers, 114.3 x 88.9 mm, 50 parts, among them J1 AudioJack, J2 Speaker, J3 UART1, J4 Pot, J6 GND, J7 DACOUT, SW1 UP, SW2 LEFT, SW3 DOWN, SW4 RGHT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

Commit message: layout
Parts:
- removed J1: AudioJack, ECE319K:Jack_3.5mm_CUI_SJ1-3523N_Horizontal
- removed U1: Adafruit ST7735R, ECE319K:adafruit_st7735r
- added G***: LOGO, ECE319K-Kaitlyn:pawn, F.Cu at (151.2, 78.2)
- added G***: LOGO, ECE319K-Kaitlyn:pawn, F.Cu at (153.8, 79.5)
- added G***: LOGO, ECE319K-Kaitlyn:pawn, F.Cu at (156.2, 78.2)
- added J5: Joystick, ECE319K:SparkfunJoystick, F.Cu at (59.4, 114.2)
- moved U4 147.9 mm to (108.4, 77.7)
- moved R12 134.2 mm to (159.2, 86.0)
- moved R13 134.0 mm to (159.2, 92.0)
- moved R14 132.0 mm to (159.2, 98.0)
- moved R15 124.9 mm to (159.2, 104.0)
- moved R18 124.0 mm to (144.8, 49.8)
- moved SW4 120.3 mm to (152.5, 109.8)
- moved U5 117.3 mm to (134.6, 40.7)
- moved D4 112.6 mm to (147.3, 42.2)
- moved SW1 106.8 mm to (141.2, 100.0)
- moved SW2 94.1 mm to (130.0, 109.8)
- moved SW3 87.4 mm to (141.2, 119.5)
- moved RV1 83.4 mm to (91.6, 116.8)
- moved J6 77.4 mm to (159.5, 55.2)
- moved TP1 77.4 mm to (151.2, 55.2)
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Connections:
- C1 pad 1: unconnected-(C1-Pad1) -> Net-(U3-FC1)
- C1 pad 2: unconnected-(C1-Pad2) -> GND
- C2 pad 1: unconnected-(C2-Pad1) -> Net-(U3-FC2)
- C2 pad 2: unconnected-(C2-Pad2) -> GND
- C3 pad 1: unconnected-(C3-Pad1) -> DACOUT
- C3 pad 2: unconnected-(C3-Pad2) -> Net-(C3-Pad2)
- C4 pad 1: unconnected-(C4-Pad1) -> +3V3
- C4 pad 2: unconnected-(C4-Pad2) -> Net-(U6-Gnd)
- D1 pad 1: unconnected-(D1-K-Pad1) -> GND
- D1 pad 2: unconnected-(D1-A-Pad2) -> Net-(D1-A)
- D2 pad 1: unconnected-(D2-K-Pad1) -> GND
- D2 pad 2: unconnected-(D2-A-Pad2) -> Net-(D2-A)
- D3 pad 1: unconnected-(D3-K-Pad1) -> GND
- D3 pad 2: unconnected-(D3-A-Pad2) -> Net-(D3-A)
- D4 pad 1: unconnected-(D4-K-Pad1) -> Net-(D4-K)
- D4 pad 2: unconnected-(D4-A-Pad2) -> Net-(D4-A)
- J2 pad 1: unconnected-(J2-Pad1) -> Net-(U3-VO1)
- J2 pad 2: unconnected-(J2-Pad2) -> Net-(U3-VO2)
- J4 pad 1: unconnected-(J4-A-Pad1) -> PB18
- J4 pad 2: unconnected-(J4-B-Pad2) -> PB18
- J7 pad 1: unconnected-(J7-A-Pad1) -> DACOUT
- J7 pad 2: unconnected-(J7-B-Pad2) -> DACOUT
- JP1 pad 1: unconnected-(JP1-A-Pad1) -> DACOUT
- JP1 pad 3: unconnected-(JP1-B-Pad3) -> PB18
- R1 pad 1: unconnected-(R1-Pad1) -> PA28
- R1 pad 2: unconnected-(R1-Pad2) -> Net-(D1-A)
- R10 pad 1: unconnected-(R10-Pad1) -> DACOUT
- R10 pad 2: unconnected-(R10-Pad2) -> PB1
- R11 pad 1: unconnected-(R11-Pad1) -> DACOUT
- R11 pad 2: unconnected-(R11-Pad2) -> PB0
- R12 pad 1: unconnected-(R12-Pad1) -> PB24
- R12 pad 2: unconnected-(R12-Pad2) -> GND
- R13 pad 1: unconnected-(R13-Pad1) -> PB23
- R13 pad 2: unconnected-(R13-Pad2) -> GND
- R14 pad 1: unconnected-(R14-Pad1) -> PA16
- R14 pad 2: unconnected-(R14-Pad2) -> GND
- R15 pad 1: unconnected-(R15-Pad1) -> PA15
- R15 pad 2: unconnected-(R15-Pad2) -> GND
- R16 pad 1: unconnected-(R16-Pad1) -> Net-(U3-VO1)
- R16 pad 2: unconnected-(R16-Pad2) -> Net-(U3-VIN)
- R17 pad 1: unconnected-(R17-Pad1) -> Net-(U3-VIN)
- R17 pad 2: unconnected-(R17-Pad2) -> Net-(C3-Pad2)
- R18 pad 1: unconnected-(R18-Pad1) -> +5V
- R18 pad 2: unconnected-(R18-Pad2) -> Net-(D4-A)
- R2 pad 1: unconnected-(R2-Pad1) -> PA27
- R2 pad 2: unconnected-(R2-Pad2) -> Net-(D2-A)
- R3 pad 1: unconnected-(R3-Pad1) -> PA26
- R3 pad 2: unconnected-(R3-Pad2) -> Net-(D3-A)
- R4 pad 1: unconnected-(R4-Pad1) -> DACOUT
- R4 pad 2: unconnected-(R4-Pad2) -> PB4
- R5 pad 1: unconnected-(R5-Pad1) -> DACOUT
- R5 pad 2: unconnected-(R5-Pad2) -> PB4
- R6 pad 1: unconnected-(R6-Pad1) -> DACOUT
- R6 pad 2: unconnected-(R6-Pad2) -> PB3
- R7 pad 1: unconnected-(R7-Pad1) -> Net-(R7-Pad1)
- R7 pad 2: unconnected-(R7-Pad2) -> PB2
- R8 pad 1: unconnected-(R8-Pad1) -> DACOUT
- R8 pad 2: unconnected-(R8-Pad2) -> Net-(R7-Pad1)
- R9 pad 1: unconnected-(R9-Pad1) -> DACOUT
- R9 pad 2: unconnected-(R9-Pad2) -> PB1
- RV1 pad 1: unconnected-(RV1-Pad1) -> GND
- RV1 pad 2: unconnected-(RV1-Pad2) -> PB18
- RV1 pad 3: unconnected-(RV1-Pad3) -> +3V3
- SW1 pad 1: unconnected-(SW1-Pad1) -> PB24
- SW1 pad 2: unconnected-(SW1-Pad2) -> +3V3
- SW2 pad 1: unconnected-(SW2-Pad1) -> PB23
- SW2 pad 2: unconnected-(SW2-Pad2) -> +3V3
- SW3 pad 1: unconnected-(SW3-Pad1) -> PA16
- SW3 pad 2: unconnected-(SW3-Pad2) -> +3V3
- SW4 pad 1: unconnected-(SW4-Pad1) -> PA15
- SW4 pad 2: unconnected-(SW4-Pad2) -> +3V3
- U3 pad 2: unconnected-(U3-FC2-Pad2) -> Net-(U3-FC2)
- U3 pad 3: unconnected-(U3-FC1-Pad3) -> Net-(U3-FC1)
- U3 pad 4: unconnected-(U3-VIN-Pad4) -> Net-(U3-VIN)
- U3 pad 5: unconnected-(U3-VO1-Pad5) -> Net-(U3-VO1)
- U3 pad 6: unconnected-(U3-Vcc-Pad6) -> +5V
- U3 pad 7: unconnected-(U3-GND-Pad7) -> GND
- U3 pad 8: unconnected-(U3-VO2-Pad8) -> Net-(U3-VO2)
- U4 pad 15: +3V3 -> Net-(U4-LED+)
- U4 pad 2: +3V3 -> Net-(U4-LED+)
- U4 pad 6: PB15 -> PB13
- U6 pad 1: unconnected-(U6-Gnd-Pad1) -> Net-(U6-Gnd)
- U6 pad 2: unconnected-(U6-Vs-Pad2) -> +3V3
- U6 pad 3: unconnected-(U6-Out-Pad3) -> PA22
Routing:
- net GND: track 0.00 -> 322.3 mm, vias 0 -> 2
- net +3V3: track 0.00 -> 312.6 mm, vias 0 -> 1
- net DACOUT: track 0.00 -> 132.1 mm
- net PA22: track 0.00 -> 109.8 mm
- net +5V: track 0.00 -> 105.1 mm
- net PA8: track 0.00 -> 100.4 mm
- net PB17: track 0.00 -> 99.4 mm
- net PA15: track 0.00 -> 97.1 mm, vias 0 -> 2
- net PA16: track 0.00 -> 97.1 mm
- net PA27: track 0.00 -> 69.0 mm
- net PB24: track 0.00 -> 68.5 mm
- net PB20: track 0.00 -> 68.5 mm, vias 0 -> 2
- net PB19: track 0.00 -> 67.0 mm, vias 0 -> 1
- net PA26: track 0.00 -> 64.5 mm
- net PB9: track 0.00 -> 63.4 mm
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Other:
- board text added: "Kaitlyn Chang Sivan Syed"
- board text removed: "Your names"

Commit message: Hai
Parts:
- removed TP1: 3.3V, ECE319K:Testpoint_1x02_P2.54mm
- added J1: Conn_01x09_Pin, Connector_PinHeader_2.54mm:PinHeader_1x09_P2.54mm_Vertical, F.Cu at (96.3, 83.2)
- added J8: Conn_01x05_Pin, Connector_PinHeader_2.54mm:PinHeader_1x05_P2.54mm_Vertical, F.Cu at (101.3, 70.4)
- U5: footprint ECE319K:DIP-16_W7.62mm -> Package_DIP:DIP-16_W7.62mm
- moved J6 1.30 mm to (159.5, 56.5)
- moved G*** 1.25 mm to (150.0, 78.2)
- moved G*** 1.25 mm to (157.5, 78.2)
- moved R5 0.70 mm to (69.0, 53.5)
- moved JP1 0.68 mm to (84.4, 112.0)
- moved J7 0.57 mm to (59.2, 72.2)
- moved SW1 0.55 mm to (141.2, 99.5)
- moved SW2 0.55 mm to (130.0, 109.2)
- moved SW3 0.55 mm to (141.2, 119.0)
- moved SW4 0.55 mm to (152.5, 109.2)
Connections:
- U5 pad 1: unconnected-(U5-1B-Pad1) -> PA8
- U5 pad 16: unconnected-(U5-1C-Pad16) -> Net-(D4-K)
- U5 pad 8: unconnected-(U5-E-Pad8) -> GND
Routing:
- net PA8: track 100.4 -> 156.0 mm
- net GND: track 322.3 -> 363.9 mm
- net +3V3: track 312.6 -> 274.6 mm, vias 1 -> 2
- net PB16: track 0.00 -> 37.6 mm
- net PB15: track 0.00 -> 33.5 mm
- net PA18: track 0.00 -> 25.1 mm
- net PA17: track 0.00 -> 23.0 mm
- net Net-(R7-Pad1): track 0.00 -> 19.5 mm
- net PB17: track 99.4 -> 117.9 mm
- net PB20: track 68.5 -> 86.1 mm
- net PB9: track 63.4 -> 73.1 mm
- net PA27: track 69.0 -> 77.0 mm
- net Net-(D4-K): track 0.00 -> 5.72 mm
- net PB23: track 62.4 -> 61.5 mm
- net DACOUT: track 132.1 -> 131.2 mm

Commit message: we did a thing
Parts:
- removed the G*** at (150.0, 78.2)
- removed the G*** at (153.8, 79.5)
- removed the G*** at (157.5, 78.2)
- removed J6: GND, ECE319K:Testpoint_1x02_P2.54mm
- added G***: LOGO, LOGO, F.Cu at (150.5, 76.6)
- added G***: LOGO, ECE319K-Kaitlyn:pawn, F.Cu at (148.2, 110.8)
- added G***: LOGO, ECE319K-Kaitlyn:pawn, F.Cu at (144.5, 112.0)
- added G***: LOGO, ECE319K-Kaitlyn:pawn, F.Cu at (140.8, 110.8)
- J1, J8: moved to B.Cu
- moved G*** 84.1 mm to (61.0, 54.9)
- turned J1 to -90 degrees
- turned J8 to -90 degrees
Routing:
- net GND: track 363.9 -> 337.8 mm
Other:
- outline, holes or cut-outs redrawn
- board text removed: "ECE319K PCB camp Spring 2025"
