File: Starter/KC47852.kicad_sch (KiCad schematic)
At the start: 49 parts, among them J1 Conn_01x09_Pin, J2 Speaker, J3 UART1, J4 Pot, J5 Joystick, J6 GND, J7 DACOUT, J8 Conn_01x05_Pin, SW1 UP, SW2 LEFT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

Commit message: we did a thing
Parts:
- removed J6: GND, ECE319K:Testpoint_1x02_P2.54mm, symbol ECE319K:Testpoint
Changed lines of the file:
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@@
 	)
 	(junction
-		(at 160.655 55.245)
-		(diameter 0)
-		(color 0 0 0 0)
-	)
-	(junction
 		(at 138.43 143.51)
 		(diameter 0)
@@
 	)
 	(junction
-		(at 164.465 55.245)
-		(diameter 0)
-		(color 0 0 0 0)
-	)
-	(junction
 		(at 46.99 153.67)
 		(diameter 0)
@@
 	(wire
 		(pts
-			(xy 160.655 55.245) (xy 164.465 55.245)
-		)
-		(stroke
-			(width 0)
-			(type default)
-		)
-	)
-	(wire
-		(pts
 			(xy 43.18 166.37) (xy 46.99 166.37)
 		)
@@
 	(wire
 		(pts
-			(xy 158.75 55.245) (xy 160.655 55.245)
-		)
-		(stroke
-			(width 0)
-			(type default)
-		)
-	)
-	(wire
-		(pts
 			(xy 46.99 147.32) (xy 49.53 147.32)
 		)
@@
 	(wire
 		(pts
-			(xy 164.465 55.245) (xy 167.64 55.245)
+			(xy 158.75 55.245) (xy 167.64 55.245)
 		)
 		(stroke
@@
 					(unit 1)
 				)
-			)
-		)
-	)
-	(symbol
-		(lib_id "ECE319K:Testpoint")
-		(at 162.56 55.245 0)
-		(unit 1)
-		(exclude_from_sim no)
-		(in_bom yes)
-		(on_board yes)
-		(dnp no)
-		(fields_autoplaced yes)
-		(property "Reference" "J6"
-			(at 162.56 50.165 0)
-			(effects
-				(font
-					(size 1.27 1.27)
-				)
-				(hide yes)
-			)
-		)
-		(property "Value" "GND"
-			(at 166.37 51.7524 0)
-			(effects
-				(font
-					(size 1.27 1.27)
-				)
-				(justify left)
-			)
-		)
-		(property "Footprint" "ECE319K:Testpoint_1x02_P2.54mm"
-			(at 162.56 49.53 0)
-			(effects
-				(font
-					(size 1.27 1.27)
-				)
-				(hide yes)
-			)
-		)
-		(property "Datasheet" "~"
-			(at 162.56 55.245 0)
-			(effects
-				(font
-					(size 1.27 1.27)
-				)
-				(hide yes)
-			)
-		)
-		(property "Description" ""
-			(at 162.56 55.245 0)
-			(effects
-				(font
-					(size 1.27 1.27)
-				)
-			)
-		)
-		(pin "1"
-		)
-		(pin "2"
-		)
-		(instances
-			(project "Starter"
-				(path "/69b823fd-c065-40ff-9bb9-c5835555f3eb"
-					(reference "J6")
-					(unit 1)
-				)
